File: HDK/brain/Connectors.kicad_sch (KiCad schematic)
At the start: 10 parts, among them J1 USB_C, J2 Can Module, J3 Can Module, J4 uC Interconnect, J5 Can Conn, J6 Can Conn, J7 Can Conn, J8 Can Conn

Commit message: updated brain
Parts:
- removed J2, J3: Can Module, symbol Connector_Generic:Conn_02x05_Odd_Even
- removed J5, J7: Can Conn, Connector_JST:JST_PH_S2B-PH-SM4-TB_1x02-1MP_P2.00mm_Horizontal, symbol Connector_Generic:Conn_01x02
- removed J6, J8: Can Conn, Connector_JST:JST_PH_B2B-PH-SM4-TB_1x02-1MP_P2.00mm_Vertical, symbol Connector_Generic:Conn_01x02
- added J304, J305: MCP251X, NVF-Kicad:Can-Module-CM251X, symbol NVF-Kicad:CM251X
- added J4: uC Interconnect, NVF-Kicad:2x04H-S, symbol Connector_Generic:Conn_02x04_Odd_Even
- added J4: DBG Connect, NVF-Kicad:2x04V-S, symbol Connector_Generic:Conn_02x04_Odd_Even
- J1: footprint (none) -> Connector_USB:USB_C_Receptacle_HRO_TYPE-C-31-M-12
- J4: footprint (none) -> NVF-Kicad:2x04H-S
- R1, R2: footprint (none) -> Resistor_SMD:R_0402_1005Metric
Connections:
- net +3V3: now also J304.10 (GND), J305.10 (GND), J4.2 (Pin_2)
- net CAN1_H: now also J304.8 (CAN_H)
- net CAN1_INT1: now also J304.2 (CAN_IRQ)
- net CAN1_L: now also J304.7 (CAN_L)
- net CAN2_H: now also J305.8 (CAN_H), J4.1 (Pin_1)
- net CAN2_INT1: now also J305.2 (CAN_IRQ)
- net CAN2_L: now also J305.7 (CAN_L), J4.2 (Pin_2)
- net GND: now also J4.5 (Pin_5), J304.9 (VCC), J305.9 (VCC), J4.4 (Pin_4), J4.4 (Pin_4), J4.5 (Pin_5); no longer J4.6 (Pin_6)
- net SPI0_CS1: now also J304.1 (~{CS})
- net SPI0_MISO: now also J304.5 (MISO)
- net SPI0_MOSI: now also J304.4 (MOSI)
- net SPI0_SCLK: now also J304.3 (SCK)
- net SPI1_CS1: now also J305.1 (~{CS})
- net SPI1_MISO: now also J305.5 (MISO)
- net SPI1_MOSI: now also J305.4 (MOSI)
- net SPI1_SCLK: now also J305.3 (SCK)
- net SWCLK: now also J4.6 (Pin_6)
- net SWDIO: now also J4.8 (Pin_8)
- net V_{IN1}: now also J4.3 (Pin_3)
- net V_{IN2}: now also J4.6 (Pin_6), J4.6 (Pin_6); no longer J4.5 (Pin_5)
- net USB_DM renamed USB_DN
- new net BOOT: J4.5 (Pin_5)
- new net IC_GP3: J4.7 (Pin_7)
- new net IC_GP4: J4.8 (Pin_8)
- new net SOF1: J304.6 (SOF)
- new net SOF2: J305.6 (SOF)
- new net UART1_RX: J4.1 (Pin_1)
- new net UART1_TX: J4.3 (Pin_3)
- new net ~{NRST}: J4.7 (Pin_7)
Other:
- company: (none) -> ScottCJX
- title: (none) -> brain
- moved on the sheet: J1, J4, R1, R2
