File: HDK/brain/Controller.kicad_sch (KiCad schematic)
At the start: 19 parts, among them U1 W25Q128JVS, U2 RP2040, Y1 12 MHz

Commit message: updated brain
Parts:
- added C11: 1u, Capacitor_SMD:C_0402_1005Metric, symbol Device:C
- added C11: 100n, Capacitor_SMD:C_0402_1005Metric, symbol Device:C
- C9: value 100n -> 1u
- U2: footprint Package_DFN_QFN:QFN-56-1EP_7x7mm_P0.4mm_EP3.2x3.2mm -> Package_DFN_QFN:QFN-56-1EP_7x7mm_P0.4mm_EP3.2x3.2mm_ThermalVias
Connections:
- net +1V1: now also C11.1
- net +3V3: now also C11.1
- net GND: now also C11.2, C11.2
- net USB_DtN: now reaches R4.2, U2.46 (USB_DM)
- net USB_DtP: now reaches R3.2, U2.47 (USB_DP)
- net SPI1_MISO renamed GP12
- net SPI1_MOSI renamed GP11
- net SPI1_SCLK renamed GP10
- net USB_DM renamed USB_DN
Other:
- company: (none) -> ScottCJX
- title: (none) -> brain
- moved on the sheet: R3, R4
