File: HDK/brain/Peripherals.kicad_sch (KiCad schematic)
At the start: 3 parts, among them U3 ADS1015IDGS, U4 ASSR-1218

Commit message: updated brain
Parts:
- removed R5: 330, symbol Device:R
- removed U3: ADS1015IDGS, Package_SO:TSSOP-10_3x3mm_P0.5mm, symbol Analog_ADC:ADS1015IDGS
- removed U4: ASSR-1218, Package_SO:SO-4_4.4x4.3mm_P2.54mm, symbol Relay_SolidState:ASSR-1218
Other:
- company: (none) -> ScottCJX
- title: (none) -> brain
