File: HDK/brain/Power.kicad_sch (KiCad schematic)
At the start: 6 parts, among them U101 LR7533-T LR

Commit message: updated brain
Parts:
- removed D501, D502, D503: D_Schottky, symbol Device:D_Schottky
- removed U101: LR7533-T LR, Package_TO_SOT_SMD:SOT-23-3, symbol Regulator_Linear:AMS1117-3.3
- added D401: BAV70, Package_TO_SOT_SMD:SOT-23, symbol Diode:BAV70
- added D402: 1N5819WS, Diode_SMD:D_SOD-323, symbol Diode:1N5819WS
- added U401: AMS1117-3.3, Package_TO_SOT_SMD:SOT-223-3_TabPin2, symbol Regulator_Linear:AMS1117-3.3
- C101, C102: value 1uF -> 4.7u; footprint (none) -> Capacitor_SMD:C_0603_1608Metric
Connections:
- net +3V3: now also U401.2 (VO)
- net GND: now also U401.1 (GND)
- net V_{IN1}: now also D401.2 (A)
- net V_{IN2}: now also D401.1 (A)
- net V_{IN}: now also D401.3 (K), D402.1 (K), U401.3 (VI)
- net V_{USB}: now also D402.2 (A)
Other:
- company: (none) -> ScottCJX
- title: (none) -> brain
