File: HDK/brain/brain.kicad_sch (KiCad schematic)
At the start: 0 parts

Commit message: updated brain
Other:
- removed sheet Peripherals
- sheet Connectors ports: added BOOT, CAN1_INT1, CAN2_INT1, UART1_RX, UART1_TX, USB_DN, ~{NRST}; removed USB_DM
- sheet Controller ports: added USB_DN; removed USB_DM
- company: (none) -> ScottCJX
- title: (none) -> brain
